File: adapter/adapter.kicad_pcb (KiCad board)
At the start: 2 copper layers, 93.5 x 50.9 mm, 64 parts, among them J1 Serial, J10 Ribbon, J11 Ribbon, J12 Ribbon, J13 serial, J14 serial, J2 Serial, J3 battery charge, J4 RGB, J5 RGB, J6 battery charge, J7 trackball, J8 trackball, J9 Ribbon, SW1 SW_SPST, SW2 SW_SPST, SW3 SW_SPDT, SW4 SW_SPDT, U1 eliteC, U2 eliteC

Commit message: routed
Parts:
- removed J13, J14: serial, Library:PinHeader_1x04_P2.54mm_Vertical
- removed J3, J6: battery charge, Library:PinHeader_1x02_P2.54mm_Vertical
- removed J4, J5: RGB, Library:header1x03
- removed J7, J8: trackball, Library:6_PinHeader
- removed JP1, JP2: Jumper_2_Open, Library:power_switch_jumper
- removed R1, R3, R5, R6: 5.1k, Library:R_1206_handsolder
- removed R2, R4: 4.7k, Library:R_1206_handsolder
- removed SW3, SW4: SW_SPDT, Library:SW_SPDT+H-MSK12C01_hor(7pin_SMD)
- removed U1, U2: eliteC, Library:Elite-C
- removed the kibuzzard-61F01957 at (121.1, 100.3)
- removed the kibuzzard-61F01957 at (121.2, 100.3)
- removed kibuzzard-620B8593 (x2): G***, kibuzzard-620B8593
- added U3: ProMicro, Library:ProMicro, B.Cu at (133.5, 83.2)
- added U4: ProMicro, Library:ProMicro, B.Cu at (177.6, 83.2)
- moved J12 5.64 mm to (183.5, 102.8)
- moved J11 4.87 mm to (177.9, 102.8)
Routing:
- net +5V: track 108.3 -> 34.9 mm
- net rgb_r: track 54.5 -> 0.00 mm
- net miso_r: track 54.1 -> 0.00 mm, vias 1 -> 0
- net mosi_r: track 49.5 -> 0.00 mm, vias 1 -> 0
- net ss_r: track 49.0 -> 0.00 mm, vias 1 -> 0
- net sc_r: track 48.4 -> 0.00 mm, vias 1 -> 0
- net rgb_l: track 40.4 -> 0.00 mm
- net sda_l: track 38.7 -> 0.00 mm, vias 1 -> 0
- net scl_l: track 36.2 -> 0.00 mm, vias 2 -> 0
- net GND: track 0.00 -> 29.5 mm
- net split_hand_r: track 28.5 -> 0.00 mm, vias 1 -> 0
- net col3_r: track 39.8 -> 12.2 mm, vias 1 -> 0
- net split_hand_l: track 26.5 -> 0.00 mm, vias 2 -> 0
- net row4_l: track 25.1 -> 0.00 mm
- net miso_l: track 24.0 -> 0.00 mm
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Other:
- board text removed: "CS"
- board text removed: "DIN"
- board text removed: "MISO"
- board text removed: "MOSI"
- board text removed: "SCL"
- board text removed: "SCLK"
- board text removed: "SDA"
