File: adapter/adapter.kicad_pcb (KiCad board)
At the start: 2 copper layers, 93.5 x 50.9 mm, 42 parts, among them J1 Serial, J10 Ribbon, J11 Ribbon, J12 Ribbon, J2 Serial, J9 Ribbon, SW1 SW_SPST, SW2 SW_SPST, U3 ProMicro, U4 ProMicro

Commit message: fixes
Routing:
- net serial_l: track 0.00 -> 22.1 mm
- net row4_l: track 0.00 -> 21.8 mm
- net Rst: track 0.00 -> 20.3 mm
- net +5V: track 34.9 -> 40.9 mm
- net GND: track 29.5 -> 35.1 mm
Changed lines of the file:
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@@
 		(pad_to_mask_clearance 0)
 		(allow_soldermask_bridges_in_footprints no)
+		(aux_axis_origin 155.47 92.52)
 		(pcbplotparams
-			(layerselection 0x00010fc_ffffffff)
+			(layerselection 0x0001000_fffffffe)
 			(plot_on_all_layers_selection 0x0000000_00000000)
 			(disableapertmacros no)
@@
 		(layer "Dwgs.User")
 	)
+	(gr_rect
+		(start 75.47 42.52)
+		(end 235.47 142.52)
+		(stroke
+			(width 0.15)
+			(type default)
+		)
+		(fill none)
+		(layer "Cmts.User")
+	)
+	(gr_line
+		(start 235.47 42.52)
+		(end 75.47 142.52)
+		(stroke
+			(width 0.15)
+			(type default)
+		)
+		(layer "Cmts.User")
+	)
+	(gr_line
+		(start 75.47 42.52)
+		(end 235.47 142.52)
+		(stroke
+			(width 0.15)
+			(type default)
+		)
+		(layer "Cmts.User")
+	)
 	(gr_arc
 		(start 173.792097 112.733917)
@@
 	)
 	(segment
+		(start 131.1 86.25)
+		(end 131.15 86.2)
+		(width 0.3)
+		(layer "B.Cu")
+		(net 2)
+	)
+	(segment
+		(start 131.15 79.57)
+		(end 125.89 74.31)
+		(width 0.3)
+		(layer "B.Cu")
+		(net 2)
+	)
+	(segment
+		(start 131.1 92.4)
+		(end 131.1 86.25)
+		(width 0.3)
+		(layer "B.Cu")
+		(net 2)
+	)
+	(segment
+		(start 131.15 86.2)
+		(end 131.15 79.57)
+		(width 0.3)
+		(layer "B.Cu")
+		(net 2)
+	)
+	(segment
 		(start 176.85 86.4)
 		(end 176.85 81.14)
@@
 	)
 	(segment
+		(start 132.689684 98.366103)
+		(end 138.481447 92.57434)
+		(width 0.3)
+		(layer "B.Cu")
+		(net 12)
+	)
+	(segment
+		(start 132.689684 102.819999)
+		(end 132.689684 98.366103)
+		(width 0.3)
+		(layer "B.Cu")
+		(net 12)
+	)
+	(segment
+		(start 138.481447 87.118553)
+		(end 141.13 84.47)
+		(width 0.3)
+		(layer "B.Cu")
+		(net 12)
+	)
+	(segment
+		(start 138.481447 92.57434)
+		(end 138.481447 87.118553)
+		(width 0.3)
+		(layer "B.Cu")
+		(net 12)
+	)
+	(segment
 		(start 134.02 104.029683)
 		(end 134.02 97.742894)
@@
 	)
 	(segment
+		(start 125.54766 71.42766)
+		(end 125.89 71.77)
+		(width 0.3)
+		(layer "B.Cu")
+		(net 29)
+	)
+	(segment
 		(start 195.231581 72.22)
 		(end 187.25 72.22)
@@
 	)
 	(segment
+		(start 120.45262 71.42766)
+		(end 125.54766 71.42766)
+		(width 0.3)
+		(layer "B.Cu")
+		(net 29)
+	)
+	(segment
 		(start 187.25 72.22)
 		(end 185.21 74.26)
@@
 	)
 	(segment
+		(start 124.46766 75.42766)
+		(end 125.89 76.85)
+		(width 0.3)
+		(layer "B.Cu")
+		(net 32)
+	)
+	(segment
+		(start 120.45262 75.42766)
+		(end 124.46766 75.42766)
+		(width 0.3)
+		(layer "B.Cu")
+		(net 32)
+	)
+	(segment
 		(start 195.898921 75.55266)
 		(end 195.898921 74.25266)
@@
 		(net 33)
 	)
+	(segment
+		(start 122.40496 70.38)
+		(end 139.74 70.38)
+		(width 0.3)
+		(layer "B.Cu")
+		(net 39)
+	)
+	(segment
+		(start 139.74 70.38)
+		(end 141.13 71.77)
+		(width 0.3)
+		(layer "B.Cu")
+		(net 39)
+	)
+	(segment
+		(start 120.45262 68.42766)
+		(end 122.40496 70.38)
+		(width 0.3)
+		(layer "B.Cu")
+		(net 39)
+	)
 	(zone
